File: PCB/kicad_boards/spikeling.kicad_pcb (KiCad board)
At the start: 2 copper layers, 55.1 x 67.7 mm, 21 parts, among them J1 D_IN1, J2 D_IN2, J3 A_IN, J4 D_OUT, J5 A_OUT, J6 Vin, J7 Arduino1-15, J8 Arduino16-30, SW1 Button

Commit message: update SMD board
Parts:
- D1: footprint LED_SMD:LED_1806_4516Metric -> LED_SMD:LED_2512_6332Metric
- moved D2 14.0 mm to (154.0, 52.0), turned to 0 degrees
- moved RV1 7.79 mm to (142.5, 116.5)
- moved D1 6.50 mm to (175.5, 117.0)
- moved RV2 6.29 mm to (142.4, 99.0)
- moved R1 6.00 mm to (175.5, 110.5)
- moved J5 5.68 mm to (187.7, 115.2)
- moved J6 5.00 mm to (162.0, 111.5)
- moved RV3 4.54 mm to (142.5, 81.5)
- moved J4 4.50 mm to (187.8, 100.5)
- moved SW1 3.50 mm to (162.0, 100.5)
- moved RV4 3.30 mm to (142.5, 64.0)
- moved J3 3.18 mm to (187.7, 85.7)
- moved J2 2.01 mm to (187.5, 70.5)
- moved J1 0.46 mm to (187.7, 55.3)
Routing:
- net Net-(D2-Pad2): track 4.00 -> 16.3 mm
- net RV1: track 49.3 -> 59.9 mm
- net Net-(C1-Pad2): track 58.8 -> 68.3 mm
- net GND: track 25.9 -> 35.3 mm, vias 3 -> 4
- net A_in: track 55.8 -> 47.9 mm, vias 0 -> 2
- net photodiode: track 57.1 -> 64.1 mm
- net Vin: track 18.7 -> 23.7 mm
- net RV4: track 29.9 -> 25.4 mm
- net D_in1: track 24.2 -> 20.2 mm
- net push_button: track 28.5 -> 32.0 mm
- net D_out: track 33.4 -> 36.3 mm
- net D_in2: track 15.2 -> 13.0 mm, vias 0 -> 1
- net RV3: track 18.5 -> 20.5 mm, vias 0 -> 1
- net RV2: track 27.2 -> 28.3 mm
Other:
- board size 55.1 x 67.7 mm -> 55.1 x 72.7 mm
- board text added: "Project hosted at: https://github.com/amchagas/spikeling"
- board text added: "Spikeling mini derivative by Chagas AM 20200716 CERN OHL-S v2.0"
