File: PCB/kicad_boards/spikeling.sch (KiCad schematic (older format))
At the start: 21 parts, among them J1 D_IN1, J2 D_IN2, J3 A_IN, J4 D_OUT, J5 A_OUT, J6 Vin, J7 Arduino1-15, J8 Arduino16-30, SW1 Button

Commit message: update smd version of board
Parts:
- BZ1: symbol Device:Buzzer -> spikeling-rescue:Buzzer-Device
- C1: symbol pspice:CAP -> spikeling-rescue:CAP-pspice
- D1: footprint LED_THT:LED_D5.0mm_Clear -> LED_SMD:LED_1806_4516Metric; symbol Device:D_Photo -> spikeling-rescue:D_Photo-Device
- D2: symbol Device:LED -> spikeling-rescue:LED-Device
- J1, J2, J3, J4, J5: symbol Connector:Conn_Coaxial -> spikeling-rescue:Conn_Coaxial-Connector
- J6: symbol Connector:Barrel_Jack -> spikeling-rescue:Barrel_Jack-Connector
- J7, J8: symbol Connector:Conn_01x15_Female -> spikeling-rescue:Conn_01x15_Female-Connector
- R1, R2, R3, R4: symbol Device:R -> spikeling-rescue:R-Device
- RV1, RV2, RV3, RV4: symbol Device:R_POT -> spikeling-rescue:R_POT-Device
- SW1: footprint Button_Switch_THT:SW_PUSH_6mm_H5mm -> Button_Switch_SMD:SW_Push_1P1T_NO_6x6mm_H9.5mm; symbol Switch:SW_Push -> spikeling-rescue:SW_Push-Switch
Changed lines of the file:
@@
 $EndDescr
 $Comp
-L Device:R_POT RV1
+L spikeling-rescue:R_POT-Device RV1
 U 1 1 5CEAF58E
 P 1650 1200
@@
 $EndComp
 $Comp
-L Device:R_POT RV2
+L spikeling-rescue:R_POT-Device RV2
 U 1 1 5CEAF60C
 P 1650 1650
@@
 $EndComp
 $Comp
-L Device:R_POT RV3
+L spikeling-rescue:R_POT-Device RV3
 U 1 1 5CEAF638
 P 1650 2100
@@
 $EndComp
 $Comp
-L Device:R_POT RV4
+L spikeling-rescue:R_POT-Device RV4
 U 1 1 5CEAF65E
 P 1650 2550
@@
 $EndComp
 $Comp
-L Device:LED D2
+L spikeling-rescue:LED-Device D2
 U 1 1 5CEAF6DF
 P 2150 5550
@@
 $EndComp
 $Comp
-L Device:R R1
+L spikeling-rescue:R-Device R1
 U 1 1 5CEAF75D
 P 1900 3900
@@
 $EndComp
 $Comp
-L Device:R R4
+L spikeling-rescue:R-Device R4
 U 1 1 5CEAF7C1
 P 2150 7050
@@
 $EndComp
 $Comp
-L Device:R R2
+L spikeling-rescue:R-Device R2
 U 1 1 5CEAF81B
 P 1650 5550
@@
 $EndComp
 $Comp
-L Device:Buzzer BZ1
+L spikeling-rescue:Buzzer-Device BZ1
 U 1 1 5CEAF8CF
 P 1600 3100
@@
 $EndComp
 $Comp
-L Switch:SW_Push SW1
+L spikeling-rescue:SW_Push-Switch SW1
 U 1 1 5CEAFDBF
 P 1600 7050
 F 0 "SW1" H 1600 7335 50  0000 C CNN
 F 1 "Button" H 1600 7244 50  0000 C CNN
-F 2 "Button_Switch_THT:SW_PUSH_6mm_H5mm" H 1600 7250 50  0001 C CNN
+F 2 "Button_Switch_SMD:SW_Push_1P1T_NO_6x6mm_H9.5mm" H 1600 7250 50  0001 C CNN
 F 3 "" H 1600 7250 50  0001 C CNN
 	1    1600 7050
@@
 $EndComp
 $Comp
-L Device:D_Photo D1
+L spikeling-rescue:D_Photo-Device D1
 U 1 1 5CEAFFD3
 P 1850 3550
 F 0 "D1" H 1800 3845 50  0000 C CNN
 F 1 "D_Photo" H 1800 3754 50  0000 C CNN
-F 2 "LED_THT:LED_D5.0mm_Clear" H 1800 3550 50  0001 C CNN
+F 2 "LED_SMD:LED_1806_4516Metric" H 1800 3550 50  0001 C CNN
 F 3 "~" H 1800 3550 50  0001 C CNN
 	1    1850 3550
@@
 $EndComp
 $Comp
-L Connector:Conn_Coaxial J4
+L spikeling-rescue:Conn_Coaxial-Connector J4
 U 1 1 5CEB0420
 P 1750 4800
@@
 $EndComp
 $Comp
-L Connector:Conn_Coaxial J3
+L spikeling-rescue:Conn_Coaxial-Connector J3
 U 1 1 5CEB049E
 P 1750 5250
@@
 	1400 7050 1150 7050
 $Comp
-L power:GND #PWR02
+L spikeling-rescue:GND-power #PWR02
 U 1 1 5CEB3156
 P 3100 3000
@@
 	5800 3950 5900 3950
 $Comp
-L power:GND #PWR022
+L spikeling-rescue:GND-power #PWR022
 U 1 1 5EBD6C21
 P 5800 2600
@@
 NoConn ~ 5900 3850
 $Comp
-L power:+5V #PWR04
+L spikeling-rescue:+5V-power #PWR04
 U 1 1 5EC8C52C
 P 1300 1800
@@
 $EndComp
 $Comp
-L power:GND #PWR012
+L spikeling-rescue:GND-power #PWR012
 U 1 1 5ECA6EC7
 P 1500 1050
@@
 	7050 3550 7250 3550
 $Comp
-L power:GND #PWR019
+L spikeling-rescue:GND-power #PWR019
 U 1 1 5ED3355E
 P 2500 7100
@@
 A_in
 $Comp
-L power:+5V #PWR023
+L spikeling-rescue:+5V-power #PWR023
 U 1 1 5ED4AD02
 P 7200 3750
@@
 	3100 3000 3100 3200
 $Comp
-L power:+5V #PWR03
+L spikeling-rescue:+5V-power #PWR03
 U 1 1 5ED6B277
 P 1150 7050
@@
 	5800 2600 5900 2600
 $Comp
-L power:GND #PWR014
+L spikeling-rescue:GND-power #PWR014
 U 1 1 5ED8CE4B
 P 2150 4600
@@
 $EndComp
 $Comp
-L power:GND #PWR018
+L spikeling-rescue:GND-power #PWR018
 U 1 1 5ED8D2CE
 P 2350 6400
@@
 $EndComp
 $Comp
-L power:GND #PWR013
+L spikeling-rescue:GND-power #PWR013
 U 1 1 5ED92A8B
 P 2100 5050
@@
 D_in1
 $Comp
-L power:GND #PWR015
+L spikeling-rescue:GND-power #PWR015
 U 1 1 5EDB3128
 P 2200 4000
@@
 $EndComp
 $Comp
-L power:GND #PWR06
+L spikeling-rescue:GND-power #PWR06
 U 1 1 5EDB4E28
 P 1350 2400
@@
 $EndComp
 $Comp
-L power:GND #PWR05
+L spikeling-rescue:GND-power #PWR05
 U 1 1 5EDB9366
 P 1350 1950
@@
 	1350 1950 1650 1950
 $Comp
-L power:GND #PWR010
+L spikeling-rescue:GND-power #PWR010
 U 1 1 5EDB9D0A
 P 1450 1500
@@
 	1500 1050 1650 1050
 $Comp
-L power:+5V #PWR09
+L spikeling-rescue:+5V-power #PWR09
 U 1 1 5EDC15D0
 P 1400 2700
@@
 	1400 2700 1650 2700
 $Comp
-L power:+5V #PWR08
+L spikeling-rescue:+5V-power #PWR08
 U 1 1 5EDC24BE
 P 1400 2250
@@
 	1300 1800 1650 1800
 $Comp
-L power:+5V #PWR07
+L spikeling-rescue:+5V-power #PWR07
 U 1 1 5EDC8C56
 P 1400 1350
@@
 	5700 3050 5900 3050
 $Comp
-L power:GND #PWR021
+L spikeling-rescue:GND-power #PWR021
 U 1 1 5EE34D61
 P 5700 2950
@@
 NoConn ~ 5900 2850
 $Comp
-L power:GND #PWR011
+L spikeling-rescue:GND-power #PWR011
 U 1 1 5EE61F1A
 P 1450 3200
@@
 	1450 3200 1500 3200
 $Comp
-L power:GND #PWR016
+L spikeling-rescue:GND-power #PWR016
 U 1 1 5EDDA56F
 P 2350 5550
@@
 	2300 5550 2350 5550
 $Comp
-L Connector:Conn_Coaxial J2
+L spikeling-rescue:Conn_Coaxial-Connector J2
 U 1 1 5CEB03E0
 P 2000 6600
@@
 $EndComp
 $Comp
-L Connector:Conn_Coaxial J1
+L spikeling-rescue:Conn_Coaxial-Connector J1
 U 1 1 5CEB038C
 P 2000 6150
@@
 	2000 5950 2350 5950
 $Comp
-L power:GND #PWR017
+L spikeling-rescue:GND-power #PWR017
 U 1 1 5ED8D9EE
 P 2350 5950
@@
 	1850 7050 2000 7050
 $Comp
-L Connector:Conn_01x15_Female J7
+L spikeling-rescue:Conn_01x15_Female-Connector J7
 U 1 1 5EB7EDA9
 P 6100 3350
@@
 	7050 3950 7250 3950
 $Comp
-L power:GND #PWR024
+L spikeling-rescue:GND-power #PWR024
 U 1 1 5EC6E46F
 P 7250 3950
@@
 	3500 1600 3400 1600
 $Comp
-L Device:R R3
+L spikeling-rescue:R-Device R3
 U 1 1 5CEAF7EB
 P 3650 1600
@@
 $EndComp
 $Comp
-L Connector:Conn_Coaxial J5
+L spikeling-rescue:Conn_Coaxial-Connector J5
 U 1 1 5CEB045C
 P 4450 1550
@@
 $EndComp
 $Comp
-L pspice:CAP C1
+L spikeling-rescue:CAP-pspice C1
 U 1 1 5CEB0504
 P 3800 1300
@@
 	3800 1550 3800 1600
 $Comp
-L power:GND #PWR01
+L spikeling-rescue:GND-power #PWR01
 U 1 1 5CEB0D1B
 P 3800 900
@@
 $EndComp
 $Comp
-L Connector:Conn_01x15_Female J8
+L spikeling-rescue:Conn_01x15_Female-Connector J8
 U 1 1 5EBB29DA
 P 6850 3350
@@
 $EndComp
 $Comp
-L power:GND #PWR020
+L spikeling-rescue:GND-power #PWR020
 U 1 1 5ED98448
 P 4450 1250
@@
 	7050 2950 7250 2950
 $Comp
-L Connector:Barrel_Jack J6
+L spikeling-rescue:Barrel_Jack-Connector J6
 U 1 1 5EB6DB43
 P 3500 3300

Commit message: modified kicad pcb
Parts:
- D1: footprint LED_SMD:LED_1806_4516Metric -> LED_SMD:LED_2512_6332Metric
Changed lines of the file:
@@
 F 0 "D1" H 1800 3845 50  0000 C CNN
 F 1 "D_Photo" H 1800 3754 50  0000 C CNN
-F 2 "LED_SMD:LED_1806_4516Metric" H 1800 3550 50  0001 C CNN
+F 2 "LED_SMD:LED_2512_6332Metric" H 1800 3550 50  0001 C CNN
 F 3 "~" H 1800 3550 50  0001 C CNN
 	1    1850 3550
